Commit message: update urdf

File: urdf/giraff_robot.urdf (robot description, URDF)
Before this commit: robot giraff_robot, 4 links, 5 joints
Links:
- added link tool_mic, mass 1.0; collision cylinder length=0.6 radius=0.5; visual cylinder length=0.6 radius=0.5
Joints:
- joint end_effector_joint: child (none) -> tool_mic

Commit message: update-28-12-23

File: urdf/giraff_robot.urdf (robot description, URDF)
Before this commit: robot giraff_robot, 5 links, 5 joints
Joints:
- removed joint neck_prismatic_joint
- added joint leg_joint: type prismatic, parent leg_link, child arm_link, origin xyz=0 0 0 rpy=0 0 0, limit lower=0.0 upper=100.0 effort=100.0 velocity=1.0
- joint base_joint: axis (none) -> 0 0 1; limit (none) -> lower=-3.1416 upper=3.1416 effort=100.0 velocity=1.0; type fixed -> revolute

Commit message: update

File: urdf/giraff_robot.urdf (robot description, URDF)
Before this commit: robot giraff_robot, 5 links, 5 joints
Links:
- added link world
Joints:
- joint base_spherical_joint: parent  -> base_link

Commit message: update

File: urdf/giraff_robot.urdf (robot description, URDF)
Before this commit: robot giraff_robot, 6 links, 5 joints
Joints:
- joint arm_joint: axis 0 0 1 -> 1 0 0
- joint base_joint: axis 0 0 1 -> 1 0 0
- joint base_spherical_joint: axis 0 0 1 -> 1 0 0
- joint end_effector_joint: axis 0 0 1 -> 0 1 0

Commit message: update

File: urdf/giraff_robot.urdf (robot description, URDF)
Before this commit: robot giraff_robot, 6 links, 5 joints
Joints:
- joint end_effector_joint: limit lower=0.0 upper=30.0 effort=100.0 velocity=1.0 -> lower=0.0 upper=0.5236 effort=100.0 velocity=1.0

Commit message: update

File: urdf/giraff_robot.urdf (robot description, URDF)
Before this commit: robot giraff_robot, 6 links, 5 joints
Joints:
- joint arm_joint: limit lower=-3.1416 upper=3.1416 effort=100.0 velocity=1.0 -> lower=-3.1416 upper=3.1416 effort=1000.0 velocity=1000.0
- joint base_joint: limit lower=-3.1416 upper=3.1416 effort=100.0 velocity=1.0 -> lower=-3.1416 upper=3.1416 effort=1000.0 velocity=1000.0
- joint base_spherical_joint: limit lower=-3.1416 upper=3.1416 effort=100.0 velocity=1.0 -> lower=-3.1416 upper=3.1416 effort=1000.0 velocity=1000.0
- joint end_effector_joint: limit lower=0.0 upper=0.5236 effort=100.0 velocity=1.0 -> lower=0.0 upper=0.5236 effort=1000.0 velocity=1000.0
- joint leg_joint: limit lower=0.0 upper=100.0 effort=100.0 velocity=1.0 -> lower=0.0 upper=100.0 effort=1000.0 velocity=1000.0
